Commit message: Update 07/23 add the usage

File: src/turtlebot_arm/turtlebot_arm_description/urdf/turtlebot_arm.urdf.xacro (robot description, xacro)
@@ -22,5 +22,5 @@
       <!-- Place the "floating" arm at the location it should be if mounted on a turtlebot,
            as pick and place and other demos assume this location -->
-      <origin xyz="0.12636 0.015 0.158"/>
+      <origin xyz="0.12636 0.015 0.208"/>
     </turtlebot_arm>
 </robot>
